Commit message: Latest config files version for CENTAURO integration week in Pisa.

File: configs/centauro/urdf/centauro_lower_body_fixed_wheels.urdf (robot description, URDF)
Before this commit: robot centauro, 49 links, 48 joints
Links:
- removed link arm1_1
- removed link arm1_2
- removed link arm1_3
- removed link arm1_4
- removed link arm1_5
- removed link arm1_6
- removed link arm1_7
- removed link arm1_8
- removed link arm2_1
- removed link arm2_2
- removed link arm2_3
- removed link arm2_4
- removed link arm2_5
- removed link arm2_6
- removed link arm2_7
- removed link arm2_8
- removed link ft_arm1
- removed link ft_arm2
- removed link imu_link
- removed link neck_1
- removed link neck_2
- removed link neck_3
- removed link torso_2
Joints:
- removed joint imu_joint
- removed joint j_arm1_1
- removed joint j_arm1_2
- removed joint j_arm1_3
- removed joint j_arm1_4
- removed joint j_arm1_5
- removed joint j_arm1_6
- removed joint j_arm1_7
- removed joint j_arm1_8
- removed joint j_arm2_1
- removed joint j_arm2_2
- removed joint j_arm2_3
- removed joint j_arm2_4
- removed joint j_arm2_5
- removed joint j_arm2_6
- removed joint j_arm2_7
- removed joint j_arm2_8
- removed joint j_ft_arm1
- removed joint j_ft_arm2
- removed joint neck_pitch
- removed joint neck_velodyne
- removed joint neck_yaw
- removed joint torso_yaw
- joint hip_yaw_1: limit lower=-1.13446401 upper=2.70526034 effort=304 velocity=8.8 -> lower=-0.78539816 upper=2.35619449 effort=304 velocity=8.8; origin xyz=0.25 0.125 -0.0566 rpy=3.14159265359 0.0 0.50709869865 -> xyz=0.225 0.125 0.11 rpy=3.14159265359 0.0 0.50709869865
- joint hip_yaw_2: limit lower=-2.70526034 upper=1.13446401 effort=304 velocity=8.8 -> lower=-2.35619449 upper=0.78539816 effort=304 velocity=8.8; origin xyz=0.25 -0.125 -0.0566 rpy=3.14159265359 0.0 -0.50709869865 -> xyz=0.225 -0.125 0.11 rpy=3.14159265359 0.0 -0.50709869865
- joint hip_yaw_3: limit lower=-2.70526034 upper=1.13446401 effort=304 velocity=8.8 -> lower=-2.35619449 upper=0.78539816 effort=304 velocity=8.8; origin xyz=-0.25 0.125 -0.0566 rpy=3.14159265359 0.0 2.63449395494 -> xyz=-0.225 0.125 0.11 rpy=3.14159265359 0.0 2.63449395494
- joint hip_yaw_4: limit lower=-1.13446401 upper=2.70526034 effort=304 velocity=8.8 -> lower=-0.78539816 upper=2.35619449 effort=304 velocity=8.8; origin xyz=-0.25 -0.125 -0.0566 rpy=3.14159265359 0.0 3.64869135224 -> xyz=-0.225 -0.125 0.11 rpy=3.14159265359 0.0 3.64869135224
- joint j_wheel_1: type continuous -> revolute
- joint j_wheel_2: type continuous -> revolute
- joint j_wheel_3: type continuous -> revolute
- joint j_wheel_4: type continuous -> revolute
- joint reference: origin xyz=0.0 0.0 0.9256 -> xyz=0.0 0.0 0.759

File: configs/centauro/urdf/centauro_lower_body_fixed_wheels_ARTURO.urdf (robot description, URDF)
Before this commit: robot centauro, 44 links, 43 joints
Links:
- removed link arm1_1
- removed link arm1_2
- removed link arm1_3
- removed link arm1_4
- removed link arm1_5
- removed link arm1_6
- removed link arm1_7
- removed link arm1_8
- removed link arm2_1
- removed link arm2_2
- removed link arm2_3
- removed link arm2_4
- removed link arm2_5
- removed link arm2_6
- removed link arm2_7
- removed link arm2_8
- removed link torso_2
- added link foot_fl, mass 0; visual box size=0.01 0.01 0.01
- added link foot_fr, mass 0; visual box size=0.01 0.01 0.01
- added link foot_hl, mass 0; visual box size=0.01 0.01 0.01
- added link foot_hr, mass 0; visual box size=0.01 0.01 0.01
Joints:
- removed joint j_arm1_1
- removed joint j_arm1_2
- removed joint j_arm1_3
- removed joint j_arm1_4
- removed joint j_arm1_5
- removed joint j_arm1_6
- removed joint j_arm1_7
- removed joint j_arm1_8
- removed joint j_arm2_1
- removed joint j_arm2_2
- removed joint j_arm2_3
- removed joint j_arm2_4
- removed joint j_arm2_5
- removed joint j_arm2_6
- removed joint j_arm2_7
- removed joint j_arm2_8
- removed joint torso_yaw
- added joint j_foot_fl: type fixed, parent ankle2_1, child foot_fl, origin xyz=0.0 0.0 0.30 rpy=0.0 0.0 0.0
- added joint j_foot_fr: type fixed, parent ankle2_2, child foot_fr, origin xyz=0.0 0.0 0.30 rpy=0.0 0.0 0.0
- added joint j_foot_hl: type fixed, parent ankle2_3, child foot_hl, origin xyz=0.0 0.0 0.30 rpy=0.0 0.0 0.0
- added joint j_foot_hr: type fixed, parent ankle2_4, child foot_hr, origin xyz=0.0 0.0 0.30 rpy=0.0 0.0 0.0
- joint j_wheel_1: type continuous -> fixed
- joint j_wheel_2: type continuous -> fixed
- joint j_wheel_3: type continuous -> fixed
- joint j_wheel_4: type continuous -> fixed

File: configs/centauro/urdf/centauro_no_head.urdf (robot description, URDF)
Before this commit: robot centauro, 36 links, 35 joints
Links:
- removed link ft_arm2
- removed link ft_foot_1
- removed link ft_foot_2
- removed link ft_foot_3
- removed link ft_foot_4
- added link ankle1_1, mass 1.2380744; collision mesh filename=package://centauro/centauro_urdf/meshes/convex_hull/ankle-p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 scale=0.001 0.001 0.001; visual mesh filename=package://centauro/centauro_urdf/meshes/ankle-pitch.stl scale=0.001 0.001 0.001
- added link ankle1_2, mass 1.2380744; collision mesh filename=package://centauro/centauro_urdf/meshes/convex_hull/ankle-p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 scale=0.001 0.001 0.001; visual mesh filename=package://centauro/centauro_urdf/meshes/ankle-pitch.stl scale=0.001 0.001 0.001
- added link ankle1_3, mass 1.2380744; collision mesh filename=package://centauro/centauro_urdf/meshes/convex_hull/ankle-p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 scale=0.001 0.001 0.001; visual mesh filename=package://centauro/centauro_urdf/meshes/ankle-pitch.stl scale=0.001 0.001 0.001
- added link ankle1_4, mass 1.2380744; collision mesh filename=package://centauro/centauro_urdf/meshes/convex_hull/ankle-p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 scale=0.001 0.001 0.001; visual mesh filename=package://centauro/centauro_urdf/meshes/ankle-pitch.stl scale=0.001 0.001 0.001
- added link ankle2_1, mass 1.1565926; collision mesh filename=package://centauro/centauro_urdf/meshes/convex_hull/ankle-y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 scale=0.001 0.001 0.001; visual mesh filename=package://centauro/centauro_urdf/meshes/ankle-yaw.stl scale=0.001 0.001 0.001
- added link ankle2_2, mass 1.1565926; collision mesh filename=package://centauro/centauro_urdf/meshes/convex_hull/ankle-y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 scale=0.001 0.001 0.001; visual mesh filename=package://centauro/centauro_urdf/meshes/ankle-yaw.stl scale=0.001 0.001 0.001
- added link ankle2_3, mass 1.1565926; collision mesh filename=package://centauro/centauro_urdf/meshes/convex_hull/ankle-y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 scale=0.001 0.001 0.001; visual mesh filename=package://centauro/centauro_urdf/meshes/ankle-yaw.stl scale=0.001 0.001 0.001
- added link ankle2_4, mass 1.1565926; collision mesh filename=package://centauro/centauro_urdf/meshes/convex_hull/ankle-y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 scale=0.001 0.001 0.001; visual mesh filename=package://centauro/centauro_urdf/meshes/ankle-yaw.stl scale=0.001 0.001 0.001
- added link arm2_8, mass 0.15; collision mesh filename=package://centauro/centauro_urdf/meshes/convex_hull/link9.s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 scale=0.001 0.001 -0.001; visual mesh filename=package://centauro/centauro_urdf/meshes/link9.stl scale=0.001 0.001 -0.001
- added link foot_fl, mass 0; visual box size=0.01 0.01 0.01
- added link foot_fr, mass 0; visual box size=0.01 0.01 0.01
- added link foot_hl, mass 0; visual box size=0.01 0.01 0.01
- added link foot_hr, mass 0; visual box size=0.01 0.01 0.01
- added link wheel_1, mass 1.7289003; collision mesh filename=package://centauro/centauro_urdf/meshes/convex_hull/wheel.s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 scale=0.001 0.001 0.001; visual mesh filename=package://centauro/centauro_urdf/meshes/wheel.stl scale=0.001 0.001 0.001
- added link wheel_2, mass 1.7289003; collision mesh filename=package://centauro/centauro_urdf/meshes/convex_hull/wheel.s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 scale=0.001 0.001 0.001; visual mesh filename=package://centauro/centauro_urdf/meshes/wheel.stl scale=0.001 0.001 0.001
- added link wheel_3, mass 1.7289003; collision mesh filename=package://centauro/centauro_urdf/meshes/convex_hull/wheel.s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 scale=0.001 0.001 0.001; visual mesh filename=package://centauro/centauro_urdf/meshes/wheel.stl scale=0.001 0.001 0.001
- added link wheel_4, mass 1.7289003; collision mesh filename=package://centauro/centauro_urdf/meshes/convex_hull/wheel.s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 scale=0.001 0.001 0.001; visual mesh filename=package://centauro/centauro_urdf/meshes/wheel.stl scale=0.001 0.001 0.001
- link arm1_1: geometry collision mesh filename=package://centauro/centauro_urdf/meshes/convex_hull/link2.s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 scale=0.001 -0.001 0.001; visual mesh filename=package://centauro/centauro_urdf/meshes/link2.stl scale=0.001 -0.001 0.001
- link arm1_2: geometry collision mesh filename=package://centauro/centauro_urdf/meshes/convex_hull/link3.s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 scale=0.001 -0.001 0.001; visual mesh filename=package://centauro/centauro_urdf/meshes/link3.stl scale=0.001 -0.001 0.001
- link arm1_3: geometry collision mesh filename=package://centauro/centauro_urdf/meshes/convex_hull/link4.s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 scale=0.001 -0.001 0.001; visual mesh filename=package://centauro/centauro_urdf/meshes/link4.stl scale=0.001 -0.001 0.001
- link arm1_4: geometry collision mesh filename=package://centauro/centauro_urdf/meshes/convex_hull/link5.s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 scale=0.001 -0.001 0.001; visual mesh filename=package://centauro/centauro_urdf/meshes/link5.stl scale=0.001 -0.001 0.001
- link arm1_5: geometry collision mesh filename=package://centauro/centauro_urdf/meshes/convex_hull/link6.s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 scale=0.001 -0.001 0.001; visual mesh filename=package://centauro/centauro_urdf/meshes/link6.stl scale=0.001 -0.001 0.001
- link arm1_6: geometry collision mesh filename=package://centauro/centauro_urdf/meshes/convex_hull/link7.s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 scale=0.001 -0.001 0.001; visual mesh filename=package://centauro/centauro_urdf/meshes/link7.stl scale=0.001 -0.001 0.001
- link arm1_7: geometry collision mesh filename=package://centauro/centauro_urdf/meshes/convex_hull/link8.s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 scale=0.001 -0.001 0.001; visual mesh filename=package://centauro/centauro_urdf/meshes/link8.stl scale=0.001 -0.001 0.001
- link arm1_8: geometry collision mesh filename=package://centauro/centauro_urdf/meshes/convex_hull/link9.s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 scale=0.001 -0.001 -0.001; visual mesh filename=package://centauro/centauro_urdf/meshes/link9.stl scale=0.001 -0.001 -0.001
- link arm2_1: geometry collision mesh filename=package://centauro/centauro_urdf/meshes/convex_hull/link2.s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 scale=0.001 0.001 0.001; visual mesh filename=package://centauro/centauro_urdf/meshes/link2.stl scale=0.001 0.001 0.001
- link arm2_2: geometry collision mesh filename=package://centauro/centauro_urdf/meshes/convex_hull/link3.s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 scale=0.001 0.001 0.001; visual mesh filename=package://centauro/centauro_urdf/meshes/link3.stl scale=0.001 0.001 0.001
- link arm2_3: geometry collision mesh filename=package://centauro/centauro_urdf/meshes/convex_hull/link4.s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 scale=0.001 0.001 0.001; visual mesh filename=package://centauro/centauro_urdf/meshes/link4.stl scale=0.001 0.001 0.001
- link arm2_4: geometry collision mesh filename=package://centauro/centauro_urdf/meshes/convex_hull/link5.s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 scale=0.001 0.001 0.001; visual mesh filename=package://centauro/centauro_urdf/meshes/link5.stl scale=0.001 0.001 0.001
- link arm2_5: geometry collision mesh filename=package://centauro/centauro_urdf/meshes/convex_hull/link6.s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 scale=0.001 0.001 0.001; visual mesh filename=package://centauro/centauro_urdf/meshes/link6.stl scale=0.001 0.001 0.001
- link arm2_6: geometry collision mesh filename=package://centauro/centauro_urdf/meshes/convex_hull/link7.s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 scale=0.001 0.001 0.001; visual mesh filename=package://centauro/centauro_urdf/meshes/link7.stl scale=0.001 0.001 0.001
- link arm2_7: geometry collision mesh filename=package://centauro/centauro_urdf/meshes/convex_hull/link8.s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 scale=0.001 0.001 0.001; visual mesh filename=package://centauro/centauro_urdf/meshes/link8.stl scale=0.001 0.001 0.001
- link hip1_1: mass 2.0 -> 1.9194403; geometry collision mesh filename=package://centauro/centauro_urdf/meshes/convex_hull/hip-yaw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 scale=0.001 0.001 0.001; visual mesh filename=package://centauro/centauro_urdf/meshes/hip-yaw.stl scale=0.001 0.001 0.001
- link hip1_2: mass 2.0 -> 1.9194403; geometry collision mesh filename=package://centauro/centauro_urdf/meshes/convex_hull/hip-yaw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 scale=0.001 0.001 0.001; visual mesh filename=package://centauro/centauro_urdf/meshes/hip-yaw.stl scale=0.001 0.001 0.001
- link hip1_3: mass 2.0 -> 1.9194403; geometry collision mesh filename=package://centauro/centauro_urdf/meshes/convex_hull/hip-yaw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 scale=0.001 0.001 0.001; visual mesh filename=package://centauro/centauro_urdf/meshes/hip-yaw.stl scale=0.001 0.001 0.001
- link hip1_4: mass 2.0 -> 1.9194403; geometry collision mesh filename=package://centauro/centauro_urdf/meshes/convex_hull/hip-yaw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 scale=0.001 0.001 0.001; visual mesh filename=package://centauro/centauro_urdf/meshes/hip-yaw.stl scale=0.001 0.001 0.001
- link hip2_1: mass 4.5 -> 2.7264471; geometry collision mesh filename=package://centauro/centauro_urdf/meshes/convex_hull/hip-pit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 scale=0.001 0.001 0.001; visual mesh filename=package://centauro/centauro_urdf/meshes/hip-pitch.stl scale=0.001 0.001 0.001
- link hip2_2: mass 4.5 -> 2.7264471; geometry collision mesh filename=package://centauro/centauro_urdf/meshes/convex_hull/hip-pit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 scale=0.001 0.001 0.001; visual mesh filename=package://centauro/centauro_urdf/meshes/hip-pitch.stl scale=0.001 0.001 0.001
- link hip2_3: mass 4.5 -> 2.7264471; geometry collision mesh filename=package://centauro/centauro_urdf/meshes/convex_hull/hip-pit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 scale=0.001 0.001 0.001; visual mesh filename=package://centauro/centauro_urdf/meshes/hip-pitch.stl scale=0.001 0.001 0.001
- link hip2_4: mass 4.5 -> 2.7264471; geometry collision mesh filename=package://centauro/centauro_urdf/meshes/convex_hull/hip-pit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 scale=0.001 0.001 0.001; visual mesh filename=package://centauro/centauro_urdf/meshes/hip-pitch.stl scale=0.001 0.001 0.001
- link knee_1: mass 3.5 -> 1.9356754; geometry collision mesh filename=package://centauro/centauro_urdf/meshes/convex_hull/knee.stl scale=0.001 0.001 0.001; visual mesh filename=package://centauro/centauro_urdf/meshes/knee.stl scale=0.001 0.001 0.001
- link knee_2: mass 3.5 -> 1.9356754; geometry collision mesh filename=package://centauro/centauro_urdf/meshes/convex_hull/knee.stl scale=0.001 0.001 0.001; visual mesh filename=package://centauro/centauro_urdf/meshes/knee.stl scale=0.001 0.001 0.001
- link knee_3: mass 3.5 -> 1.9356754; geometry collision mesh filename=package://centauro/centauro_urdf/meshes/convex_hull/knee.stl scale=0.001 0.001 0.001; visual mesh filename=package://centauro/centauro_urdf/meshes/knee.stl scale=0.001 0.001 0.001
- link knee_4: mass 3.5 -> 1.9356754; geometry collision mesh filename=package://centauro/centauro_urdf/meshes/convex_hull/knee.stl scale=0.001 0.001 0.001; visual mesh filename=package://centauro/centauro_urdf/meshes/knee.stl scale=0.001 0.001 0.001
- link pelvis: mass 25.0 -> 24.190945; geometry collision mesh filename=package://centauro/centauro_urdf/meshes/convex_hull/pelvis.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 scale=0.001 0.001 0.001; visual mesh filename=package://centauro/centauro_urdf/meshes/pelvis.stl scale=0.001 0.001 0.001
- link torso_2: geometry collision mesh filename=package://centauro/centauro_urdf/meshes/convex_hull/link1.s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 scale=0.001 0.001 0.001; visual mesh filename=package://centauro/centauro_urdf/meshes/link1.stl scale=0.001 0.001 0.001
Joints:
- removed joint ft_foot_1_joint
- removed joint ft_foot_2_joint
- removed joint ft_foot_3_joint
- removed joint ft_foot_4_joint
- removed joint j_ft_arm2
- added joint ankle_pitch_1: type revolute, parent knee_1, child ankle1_1, origin xyz=0.2 0.0 -0.10015 rpy=3.14159265359 0.0 0.0, axis 0 0 1, limit lower=-2.61799388 upper=2.61799388 effort=147 velocity=8.1
- added joint ankle_pitch_2: type revolute, parent knee_2, child ankle1_2, origin xyz=0.2 0.0 -0.10015 rpy=3.14159265359 0.0 0.0, axis 0 0 1, limit lower=-2.61799388 upper=2.61799388 effort=147 velocity=8.1
- added joint ankle_pitch_3: type revolute, parent knee_3, child ankle1_3, origin xyz=0.2 0.0 -0.10015 rpy=3.14159265359 0.0 0.0, axis 0 0 1, limit lower=-2.61799388 upper=2.61799388 effort=147 velocity=8.1
- added joint ankle_pitch_4: type revolute, parent knee_4, child ankle1_4, origin xyz=0.2 0.0 -0.10015 rpy=3.14159265359 0.0 0.0, axis 0 0 1, limit lower=-2.61799388 upper=2.61799388 effort=147 velocity=8.1
- added joint ankle_yaw_1: type revolute, parent ankle1_1, child ankle2_1, origin xyz=0.0 0.0 0.0 rpy=1.57079632679 0.0 1.57079632679, axis 0 0 1, limit lower=-2.79252680 upper=2.79252680 effort=35 velocity=20.0
- added joint ankle_yaw_2: type revolute, parent ankle1_2, child ankle2_2, origin xyz=0.0 0.0 0.0 rpy=1.57079632679 0.0 1.57079632679, axis 0 0 1, limit lower=-2.79252680 upper=2.79252680 effort=35 velocity=20.0
- added joint ankle_yaw_3: type revolute, parent ankle1_3, child ankle2_3, origin xyz=0.0 0.0 0.0 rpy=1.57079632679 0.0 1.57079632679, axis 0 0 1, limit lower=-2.79252680 upper=2.79252680 effort=35 velocity=20.0
- added joint ankle_yaw_4: type revolute, parent ankle1_4, child ankle2_4, origin xyz=0.0 0.0 0.0 rpy=1.57079632679 0.0 1.57079632679, axis 0 0 1, limit lower=-2.79252680 upper=2.79252680 effort=35 velocity=20.0
- added joint j_arm2_8: type fixed, parent arm2_7, child arm2_8, origin xyz=0.0 0.0 -0.0405 rpy=0.0 3.14159265359 -1.5707963268, axis 1 0 0, limit lower=0.0 upper=0 effort=0 velocity=0
- added joint j_foot_fl: type fixed, parent ankle2_1, child foot_fl, origin xyz=0.0 0.0 0.30 rpy=0.0 0.0 0.0
- added joint j_foot_fr: type fixed, parent ankle2_2, child foot_fr, origin xyz=0.0 0.0 0.30 rpy=0.0 0.0 0.0
- added joint j_foot_hl: type fixed, parent ankle2_3, child foot_hl, origin xyz=0.0 0.0 0.30 rpy=0.0 0.0 0.0
- added joint j_foot_hr: type fixed, parent ankle2_4, child foot_hr, origin xyz=0.0 0.0 0.30 rpy=0.0 0.0 0.0
- added joint j_wheel_1: type revolute, parent ankle2_1, child wheel_1, origin xyz=0.0 0.00085 0.235 rpy=1.57079632679 0.0 0.0, axis 0 0 1, limit lower=-1000000000000000 upper=1000000000000000 effort=35 velocity=20.0
- added joint j_wheel_2: type revolute, parent ankle2_2, child wheel_2, origin xyz=0.0 0.00085 0.235 rpy=1.57079632679 0.0 0.0, axis 0 0 1, limit lower=-1000000000000000 upper=1000000000000000 effort=35 velocity=20.0
- added joint j_wheel_3: type revolute, parent ankle2_3, child wheel_3, origin xyz=0.0 0.00085 0.235 rpy=1.57079632679 0.0 0.0, axis 0 0 1, limit lower=-1000000000000000 upper=1000000000000000 effort=35 velocity=20.0
- added joint j_wheel_4: type revolute, parent ankle2_4, child wheel_4, origin xyz=0.0 0.00085 0.235 rpy=1.57079632679 0.0 0.0, axis 0 0 1, limit lower=-1000000000000000 upper=1000000000000000 effort=35 velocity=20.0
- joint hip_pitch_1: axis 0 -1 0 -> 0 0 1; limit lower=-3.14 upper=3.14 effort=330 velocity=6.5 -> lower=-2.09439510 upper=2.09439510 effort=304 velocity=8.8; origin xyz=0.0 0.0 -0.2 -> xyz=0.0 0.0 0.059 rpy=1.57079632679 0.0 0.50709869865
- joint hip_pitch_2: axis 0 1 0 -> 0 0 1; limit lower=-3.14 upper=3.14 effort=330 velocity=6.5 -> lower=-2.09439510 upper=2.09439510 effort=304 velocity=8.8; origin xyz=0.0 0.0 -0.2 -> xyz=0.0 0.0 0.059 rpy=1.57079632679 0.0 2.63449395494
- joint hip_pitch_3: axis 0 1 0 -> 0 0 1; limit lower=-3.14 upper=3.14 effort=330 velocity=6.5 -> lower=-2.09439510 upper=2.09439510 effort=304 velocity=8.8; origin xyz=0.0 0.0 -0.2 -> xyz=0.0 0.0 0.059 rpy=1.57079632679 0.0 2.63449395494
- joint hip_pitch_4: axis 0 -1 0 -> 0 0 1; limit lower=-3.14 upper=3.14 effort=330 velocity=6.5 -> lower=-2.09439510 upper=2.09439510 effort=304 velocity=8.8; origin xyz=0.0 0.0 -0.2 -> xyz=0.0 0.0 0.059 rpy=1.57079632679 0.0 0.50709869865
- joint hip_yaw_1: axis 0 0 -1 -> 0 0 1; limit lower=-2.09 upper=2.09 effort=147 velocity=6.5 -> lower=-0.78539816 upper=2.35619449 effort=304 velocity=8.8; origin xyz=0.3 0.15 0 rpy=0 0 1.5707963268 -> xyz=0.225 0.125 0.11 rpy=3.14159265359 0.0 0.50709869865
- joint hip_yaw_2: limit lower=-2.09 upper=2.09 effort=147 velocity=6.5 -> lower=-2.35619449 upper=0.78539816 effort=304 velocity=8.8; origin xyz=0.3 -0.15 0 rpy=0 0 1.5707963268 -> xyz=0.225 -0.125 0.11 rpy=3.14159265359 0.0 -0.50709869865
- joint hip_yaw_3: limit lower=-2.09 upper=2.09 effort=147 velocity=6.5 -> lower=-2.35619449 upper=0.78539816 effort=304 velocity=8.8; origin xyz=-0.3 -0.15 0 rpy=0 0 1.5707963268 -> xyz=-0.225 0.125 0.11 rpy=3.14159265359 0.0 2.63449395494
- joint hip_yaw_4: axis 0 0 -1 -> 0 0 1; limit lower=-2.09 upper=2.09 effort=147 velocity=6.5 -> lower=-0.78539816 upper=2.35619449 effort=304 velocity=8.8; origin xyz=-0.3 0.15 0 rpy=0 0 1.5707963268 -> xyz=-0.225 -0.125 0.11 rpy=3.14159265359 0.0 3.64869135224
- joint knee_pitch_1: axis 0 -1 0 -> 0 0 1; limit lower=-3.14 upper=3.14 effort=330 velocity=6.5 -> lower=-2.61799388 upper=2.61799388 effort=304 velocity=8.8; origin xyz=0.0 0.0 -0.35 -> xyz=0.0 0.3 -0.0036 rpy=3.14159265359 0.0 1.57079632679
- joint knee_pitch_2: axis 0 1 0 -> 0 0 1; limit lower=-3.14 upper=3.14 effort=330 velocity=6.5 -> lower=-2.61799388 upper=2.61799388 effort=304 velocity=8.8; origin xyz=0.0 0.0 -0.35 -> xyz=0.0 0.3 -0.0036 rpy=3.14159265359 0.0 1.57079632679
- joint knee_pitch_3: axis 0 1 0 -> 0 0 1; limit lower=-3.14 upper=3.14 effort=330 velocity=6.5 -> lower=-2.61799388 upper=2.61799388 effort=304 velocity=8.8; origin xyz=0.0 0.0 -0.35 -> xyz=0.0 0.3 -0.0036 rpy=3.14159265359 0.0 1.57079632679
- joint knee_pitch_4: axis 0 -1 0 -> 0 0 1; limit lower=-3.14 upper=3.14 effort=330 velocity=6.5 -> lower=-2.61799388 upper=2.61799388 effort=304 velocity=8.8; origin xyz=0.0 0.0 -0.35 -> xyz=0.0 0.3 -0.0036 rpy=3.14159265359 0.0 1.57079632679
- joint reference: origin xyz=0.0 0.0 0.85 -> xyz=0.0 0.0 0.759
- joint torso_yaw: origin xyz=0.3 0.0 0.1 -> xyz=0.175 0.0 0.36
